File: PCB/tamagotchi/tamagotchi_panel_rounded.kicad_pcb (KiCad board)
At the start: 2 copper layers, 37.5 x 66 mm, 21 parts, among them J1 Programming port, J2 Conn_01x01_Female, J3 Conn_01x01_Female, J4 Conn_01x01_Male, J5 Conn_01x01_Male, SW1 Main Button, SW2 SW_Push, U1 ATtiny85V-10P, U2 OLED

Commit message: optimized animation system
Parts:
- G***: moved to B.Cu
- moved G*** 3.26 mm to (42.5, 60.8), turned to 180 degrees
