File: PCB/tamagotchi/tamagotchi_depanelled.kicad_sch (KiCad schematic)
At the start: 13 parts, among them J1 Programming port, J2 Conn_01x01_Female, J3 Conn_01x01_Female, J6 Conn_01x01_Female, SW1 Main Button, SW2 SW_Push, U1 ATtiny85V-10P, U2 OLED

Commit message: idk
Parts:
- removed D3: LED, LED_THT:LED_D1.8mm_W3.3mm_H2.4mm, symbol Device:LED
Connections:
- net ISP MISO: now also D2.2 (A); no longer J6.1 (Pin_1)
- net ISP RESET: no longer D2.2 (A)
- no-connect marks 0 -> 1
